File: Micro-XTCF.sch (KiCad schematic (older format))
At the start: 21 parts, among them P1 CF_CARD, P2 IDE LED, SW1 ROM Enable, SW2 ROM Write Enable, U1 28C64, U2 ATF16V8B, U5 74HCT04

Commit message: Rev 1.1
Added two decouple capacitors (100nF and 22uF) on the vcc line of the cf, some cf's requires a pump when they start, thanks @arananet for the suggestion.

Added gerbers to the github project.
Parts:
- added C6: 22uF, Capacitor_SMD:C_1206_3216Metric_Pad1.33x1.80mm_HandSolder, symbol Micro-XTCF-rescue:C-Device-xt-cf-mini-rescue
- added C7: 0.1uF, Capacitor_SMD:C_1206_3216Metric_Pad1.33x1.80mm_HandSolder, symbol Micro-XTCF-rescue:C-Device-xt-cf-mini-rescue
- BUS1: symbol Micro-XTCF-rescue:BUSPC_DEV-xt-cf-rescue-xt-cf-mini-rescue-Micro-XTCF-rescue -> Micro-XTCF-rescue:BUSPC_DEV-xt-cf-rescue-xt-cf-mini-rescue
- C1, C2, C3: symbol Micro-XTCF-rescue:C-Device-xt-cf-mini-rescue-Micro-XTCF-rescue -> Micro-XTCF-rescue:C-Device-xt-cf-mini-rescue
- C4, C5: symbol Micro-XTCF-rescue:CP-Device-xt-cf-mini-rescue-Micro-XTCF-rescue -> Micro-XTCF-rescue:CP-Device-xt-cf-mini-rescue
- D1: symbol Micro-XTCF-rescue:LED-Device-xt-cf-mini-rescue-Micro-XTCF-rescue -> Micro-XTCF-rescue:LED-Device-xt-cf-mini-rescue
- P1: symbol Micro-XTCF-rescue:CF_CARD-xt-cf-rescue-xt-cf-mini-rescue-Micro-XTCF-rescue -> Micro-XTCF-rescue:CF_CARD-xt-cf-rescue-xt-cf-mini-rescue
- P2: symbol Micro-XTCF-rescue:CONN_2-xt-cf-rescue-xt-cf-mini-rescue-Micro-XTCF-rescue -> Micro-XTCF-rescue:CONN_2-xt-cf-rescue-xt-cf-mini-rescue
- R1, R2, R3, R4, R5, R6, R7: symbol Micro-XTCF-rescue:R-xt-cf-rescue-xt-cf-mini-rescue-Micro-XTCF-rescue -> Micro-XTCF-rescue:R-xt-cf-rescue-xt-cf-mini-rescue
- SW1, SW2: symbol Micro-XTCF-rescue:SW_SPDT-Switch-xt-cf-mini-rescue-Micro-XTCF-rescue -> Micro-XTCF-rescue:SW_SPDT-Switch-xt-cf-mini-rescue
- U1: symbol Micro-XTCF-rescue:28C64-xt-cf-rescue-xt-cf-mini-rescue-Micro-XTCF-rescue -> Micro-XTCF-rescue:28C64-xt-cf-rescue-xt-cf-mini-rescue
- U2: symbol Micro-XTCF-rescue:GAL16V8-Logic_Programmable-xt-cf-mini-rescue-Micro-XTCF-rescue -> Micro-XTCF-rescue:GAL16V8-Logic_Programmable-xt-cf-mini-rescue
- U5: symbol Micro-XTCF-rescue:74LS04-xt-cf-rescue-xt-cf-mini-rescue-Micro-XTCF-rescue -> Micro-XTCF-rescue:74LS04-xt-cf-rescue-xt-cf-mini-rescue
Connections:
- net GND: now also C6.2, C7.2
- net VCC: now also C6.1, C7.1
Other:
- moved on the sheet: C1, C2, C3, C4, C5
